Commit message: updated vtol nav, description and robots config

File: src/vtol_dron_description/urdf/vtol_dron.urdf (robot description, URDF)
Before this commit: robot vtol_dron, 6 links, 5 joints
Links:
- link base_link: geometry collision mesh filename=file:///home/dmitriyb51/swarm_robots_ws/install/vtol_dron_d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 scale=0.001 0.001 0.001; visual mesh filename=file:///home/dmitriyb51/swarm_robots_ws/install/vtol_dron_d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 scale=0.001 0.001 0.001
- link front_left_propeller_1_1: geometry collision mesh filename=file:///home/dmitriyb51/swarm_robots_ws/install/vtol_dron_d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 scale=0.001 0.001 0.001; visual mesh filename=file:///home/dmitriyb51/swarm_robots_ws/install/vtol_dron_d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 scale=0.001 0.001 0.001
- link mechanism__1_1: geometry collision mesh filename=file:///home/dmitriyb51/swarm_robots_ws/install/vtol_dron_d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 scale=0.001 0.001 0.001; visual mesh filename=file:///home/dmitriyb51/swarm_robots_ws/install/vtol_dron_d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 scale=0.001 0.001 0.001
- link rear_left_propeller_1_1: geometry collision mesh filename=file:///home/dmitriyb51/swarm_robots_ws/install/vtol_dron_d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 scale=0.001 0.001 0.001; visual mesh filename=file:///home/dmitriyb51/swarm_robots_ws/install/vtol_dron_d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 scale=0.001 0.001 0.001
- link rear_right__1_1: geometry collision mesh filename=file:///home/dmitriyb51/swarm_robots_ws/install/vtol_dron_d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 scale=0.001 0.001 0.001; visual mesh filename=file:///home/dmitriyb51/swarm_robots_ws/install/vtol_dron_d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 scale=0.001 0.001 0.001
- link right_front_propeller_1_1: geometry collision mesh filename=file:///home/dmitriyb51/swarm_robots_ws/install/vtol_dron_d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 scale=0.001 0.001 0.001; visual mesh filename=file:///home/dmitriyb51/swarm_robots_ws/install/vtol_dron_d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 scale=0.001 0.001 0.001
